Commit message: update

File: open_manipulator_7dof_description/urdf/open_manipulator_7dof_with_gripper.urdf.xacro (robot description, xacro)
@@ -4,5 +4,5 @@
   <link name="link1">
     <visual>
-      <origin xyz="0 0 0" rpy="0 0 0"/>
+      <origin xyz="0 0 0" rpy="${pi/2} 0 ${pi/2}"/>
       <geometry>
         <mesh filename="package://open_manipulator_7dof_description/meshes/link1.stl" scale="0.001 0.001 0.001"/>
@@ -11,5 +11,5 @@
     </visual>
     <collision>
-      <origin xyz="0 0 0" rpy="0 0 0"/>
+      <origin xyz="0 0 0" rpy="${pi/2} 0 ${pi/2}"/>
       <geometry>
         <mesh filename="package://open_manipulator_7dof_description/meshes/link1.stl" scale="0.001 0.001 0.001"/>
@@ -27,5 +27,5 @@
     <parent link="link1"/>
     <child link="link2"/>
-    <origin xyz="0.0 0.0 0.126" rpy="0 0 0"/>
+    <origin xyz="0.0 0.0 0.124" rpy="0 0 0"/>
     <axis xyz="0 0 1"/>
     <limit velocity="6.5" effort="1000" lower="${-pi*0.5}" upper="${pi*0.5}" />
@@ -35,5 +35,5 @@
   <link name="link2">
     <visual>
-      <origin xyz="0 0 0" rpy="0 0 0"/>
+      <origin xyz="0 0 0" rpy="${pi/2} 0 ${pi/2}"/>
       <geometry>
         <mesh filename="package://open_manipulator_7dof_description/meshes/link2.stl" scale="0.001 0.001 0.001"/>
@@ -42,5 +42,5 @@
     </visual>
     <collision>
-      <origin xyz="0 0 0" rpy="0 0 0"/>
+      <origin xyz="0 0 0" rpy="${pi/2} 0 ${pi/2}"/>
       <geometry>
         <mesh filename="package://open_manipulator_7dof_description/meshes/link2.stl" scale="0.001 0.001 0.001"/>
@@ -59,5 +59,5 @@
     <parent link="link2"/>
     <child link="link3"/>
-    <origin xyz="0.0 0.069 0.033" rpy="0 0 0"/>
+    <origin xyz="0.0 0.0 0.033" rpy="0 0 0"/>
     <axis xyz="0 1 0"/>
     <limit velocity="6.5" effort="1000" lower="${-pi*0.5}" upper="${pi*0.5}" />
@@ -67,5 +67,5 @@
   <link name="link3">
     <visual>
-      <origin xyz="0 0 0" rpy="0 0 0"/>
+      <origin xyz="0 -0.069 0.0" rpy="${pi/2} 0 ${pi/2}"/>
       <geometry>
         <mesh filename="package://open_manipulator_7dof_description/meshes/link3.stl" scale="0.001 0.001 0.001"/>
@@ -74,5 +74,5 @@
     </visual>
     <collision>
-      <origin xyz="0 0 0" rpy="0 0 0"/>
+      <origin xyz="0 -0.069 0.0" rpy="${pi/2} 0 ${pi/2}"/>
       <geometry>
         <mesh filename="package://open_manipulator_7dof_description/meshes/link3.stl" scale="0.001 0.001 0.001"/>
@@ -91,6 +91,6 @@
     <parent link="link3"/>
     <child link="link4"/>
-    <origin xyz="0.03000 -0.01150 0.26400" rpy="0 0 0"/>
-    <axis xyz="0 1 0"/>
+    <origin xyz="0.0 0.0 0.195" rpy="0 0 0"/>
+    <axis xyz="0 0 1"/>
     <limit velocity="6.5" effort="1000" lower="${-pi*0.5}" upper="${pi*0.5}" />
     <dynamics damping="0.7"/>
@@ -99,5 +99,5 @@
   <link name="link4">
     <visual>
-      <origin xyz="0 0 0" rpy="0 0 0"/>
+      <origin xyz="0 0 0" rpy="${pi/2} 0 ${pi/2}"/>
       <geometry>
         <mesh filename="package://open_manipulator_7dof_description/meshes/link4.stl" scale="0.001 0.001 0.001"/>
@@ -106,5 +106,5 @@
     </visual>
     <collision>
-      <origin xyz="0 0 0" rpy="0 0 0"/>
+      <origin xyz="0 0 0" rpy="${pi/2} 0 ${pi/2}"/>
       <geometry>
         <mesh filename="package://open_manipulator_7dof_description/meshes/link4.stl" scale="0.001 0.001 0.001"/>
@@ -123,6 +123,6 @@
     <parent link="link4"/>
     <child link="link5"/>
-    <origin xyz="0.19500 -0.05750 0.03000" rpy="0 0 0"/>
-    <axis xyz="1 0 0"/>
+    <origin xyz="0.0 0.0 0.069" rpy="0 0 0"/>
+    <axis xyz="0 1 0"/>
     <limit velocity="6.5" effort="1000" lower="${-pi*0.5}" upper="${pi*0.5}" />
     <dynamics damping="0.7"/>
@@ -131,5 +131,5 @@
   <link name="link5">
     <visual>
-      <origin xyz="0 0 0" rpy="0 0 0"/>
+      <origin xyz="0 -0.057 0" rpy="${pi/2} 0 ${pi/2}"/>
       <geometry>
         <mesh filename="package://open_manipulator_7dof_description/meshes/link5.stl" scale="0.001 0.001 0.001"/>
@@ -138,5 +138,5 @@
     </visual>
     <collision>
-      <origin xyz="0 0 0" rpy="0 0 0"/>
+      <origin xyz="0 -0.057 0" rpy="${pi/2} 0 ${pi/2}"/>
       <geometry>
         <mesh filename="package://open_manipulator_7dof_description/meshes/link5.stl" scale="0.001 0.001 0.001"/>
@@ -155,6 +155,6 @@
     <parent link="link5"/>
     <child link="link6"/>
-    <origin xyz="0.06300 0.04500 0.00000" rpy="0 0 0"/>
-    <axis xyz="0 1 0"/>
+    <origin xyz="0.0 0.0 0.195" rpy="0 0 0"/>
+    <axis xyz="0 0 1"/>
     <limit velocity="6.5" effort="1000" lower="${-pi*0.5}" upper="${pi*0.5}" />
     <dynamics damping="0.7"/>
@@ -163,5 +163,5 @@
   <link name="link6">
     <visual>
-      <origin xyz="0 0 0" rpy="0 0 0"/>
+      <origin xyz="0 0 0" rpy="${pi/2} 0 ${pi/2}"/>
       <geometry>
         <mesh filename="package://open_manipulator_7dof_description/meshes/link6.stl" scale="0.001 0.001 0.001"/>
@@ -170,5 +170,5 @@
     </visual>
     <collision>
-      <origin xyz="0 0 0" rpy="0 0 0"/>
+      <origin xyz="0 0 0" rpy="${pi/2} 0 ${pi/2}"/>
       <geometry>
         <mesh filename="package://open_manipulator_7dof_description/meshes/link6.stl" scale="0.001 0.001 0.001"/>
@@ -186,7 +186,39 @@
   <joint name="joint6" type="revolute">
     <parent link="link6"/>
+    <child link="link7"/>
+    <origin xyz="0.0 0.0 0.063" rpy="0 0 0"/>
+    <axis xyz="0 1 0"/>
+    <limit velocity="6.5" effort="1000" lower="${-pi*0.5}" upper="${pi*0.5}" />
+    <dynamics damping="0.7"/>
+  </joint>
+  <!-- link 7 -->
+  <link name="link7">
+    <visual>
+      <origin xyz="0 -0.045 0" rpy="${pi/2} 0 ${pi/2}"/>
+      <geometry>
+        <mesh filename="package://open_manipulator_7dof_description/meshes/link7.stl" scale="0.001 0.001 0.001"/>
+      </geometry>
+      <material name="grey"/>
+    </visual>
+    <collision>
+      <origin xyz="0 -0.045 0" rpy="${pi/2} 0 ${pi/2}"/>
+      <geometry>
+        <mesh filename="package://open_manipulator_7dof_description/meshes/link7.stl" scale="0.001 0.001 0.001"/>
+      </geometry>
+    </collision>
+    <inertial>
+      <origin xyz="0.06831 -0.04457 0.00000" rpy="0 0 0"/>
+      <!--<origin xyz="-0.05469 0.00043 0.00000" rpy="0 0 0"/>-->
+      <mass value="0.43273"/>
+      <inertia ixx="1.0" ixy="0.0" ixz="0.0" iyy="1.0" iyz="0.0" izz="1.0" />
+      <!--<inertia ixx="0.00021512" ixy="0.00001009" ixz="0.00000000" iyy="0.00042827" iyz="0.00000000" izz="0.00051436" />-->
+    </inertial>
+  </link>
+  <!-- Joint 7 -->
+  <joint name="joint7" type="revolute">
+    <parent link="link7"/>
     <child link="end_link"/>
-    <origin xyz="0.12300 -0.04500 0.00000" rpy="0 0 0"/>
-    <axis xyz="1 0 0"/>
+    <origin xyz="0.0 0.0 0.12300" rpy="0 0 0"/>
+    <axis xyz="0 0 1"/>
     <limit velocity="6.5" effort="1000" lower="${-pi*0.5}" upper="${pi*0.5}" />
     <dynamics damping="0.7"/>
@@ -195,5 +227,5 @@
   <link name="end_link">
     <visual>
-      <origin xyz="0.0 0.0 0.0" rpy="0 0 0" />
+      <origin xyz="0.0 0.0 0.0" rpy="0 -${pi/2} -${pi/2}" />
       <geometry>
         <mesh filename="package://open_manipulator_7dof_description/meshes/end_link.stl" scale="0.001 0.001 0.001"/>
@@ -202,5 +234,5 @@
     </visual>
     <collision>
-      <origin xyz="0.0 0.0 0.0" rpy="0 0 0" />
+      <origin xyz="0.0 0.0 0.0" rpy="0 -${pi/2} -${pi/2}" />
       <geometry>
         <mesh filename="package://open_manipulator_7dof_description/meshes/end_link.stl" scale="0.001 0.001 0.001"/>
@@ -218,5 +250,5 @@
     <parent link="end_link"/>
     <child link="gripper_main_link"/>
-    <origin xyz="0.007 0.0 0.0" rpy="0 0 0" />
+    <origin xyz="0.0 0.0 0.00625" rpy="0 -${pi/2} 0" />
   </joint>
   <!-- gripper main link -->
