Commit message: 7DOF

File: open_manipulator_7dof_description/urdf/open_manipulator_7dof.urdf.xacro (robot description, xacro)
@@ -4,5 +4,5 @@
   <link name="link1">
     <visual>
-      <origin xyz="0 0 0" rpy="${pi/2} 0 ${pi/2}"/>
+      <origin xyz="0 0 0" rpy="0 0 0"/>
       <geometry>
         <mesh filename="package://open_manipulator_7dof_description/meshes/link1.stl" scale="0.001 0.001 0.001"/>
@@ -11,5 +11,5 @@
     </visual>
     <collision>
-      <origin xyz="0 0 0" rpy="${pi/2} 0 ${pi/2}"/>
+      <origin xyz="0 0 0" rpy="0 0 0"/>
       <geometry>
         <mesh filename="package://open_manipulator_7dof_description/meshes/link1.stl" scale="0.001 0.001 0.001"/>
@@ -27,5 +27,5 @@
     <parent link="link1"/>
     <child link="link2"/>
-    <origin xyz="0.0 0.0 0.124" rpy="0 0 0"/>
+    <origin xyz="0.0 0.0 0.126" rpy="0 0 0"/>
     <axis xyz="0 0 1"/>
     <limit velocity="6.5" effort="1000" lower="${-pi*0.5}" upper="${pi*0.5}" />
@@ -35,5 +35,5 @@
   <link name="link2">
     <visual>
-      <origin xyz="0 0 0" rpy="${pi/2} 0 ${pi/2}"/>
+      <origin xyz="0 0 0" rpy="0 0 0"/>
       <geometry>
         <mesh filename="package://open_manipulator_7dof_description/meshes/link2.stl" scale="0.001 0.001 0.001"/>
@@ -42,5 +42,5 @@
     </visual>
     <collision>
-      <origin xyz="0 0 0" rpy="${pi/2} 0 ${pi/2}"/>
+      <origin xyz="0 0 0" rpy="0 0 0"/>
       <geometry>
         <mesh filename="package://open_manipulator_7dof_description/meshes/link2.stl" scale="0.001 0.001 0.001"/>
@@ -59,5 +59,5 @@
     <parent link="link2"/>
     <child link="link3"/>
-    <origin xyz="0.0 0.0 0.033" rpy="0 0 0"/>
+    <origin xyz="0.0 0.069 0.033" rpy="0 0 0"/>
     <axis xyz="0 1 0"/>
     <limit velocity="6.5" effort="1000" lower="${-pi*0.5}" upper="${pi*0.5}" />
@@ -67,5 +67,5 @@
   <link name="link3">
     <visual>
-      <origin xyz="0 -0.069 0.0" rpy="${pi/2} 0 ${pi/2}"/>
+      <origin xyz="0 0 0" rpy="0 0 0"/>
       <geometry>
         <mesh filename="package://open_manipulator_7dof_description/meshes/link3.stl" scale="0.001 0.001 0.001"/>
@@ -74,5 +74,5 @@
     </visual>
     <collision>
-      <origin xyz="0 -0.069 0.0" rpy="${pi/2} 0 ${pi/2}"/>
+      <origin xyz="0 0 0" rpy="0 0 0"/>
       <geometry>
         <mesh filename="package://open_manipulator_7dof_description/meshes/link3.stl" scale="0.001 0.001 0.001"/>
@@ -91,5 +91,5 @@
     <parent link="link3"/>
     <child link="link4"/>
-    <origin xyz="0.0 0.0 0.195" rpy="0 0 0"/>
+    <origin xyz="0.0 -0.069 0.195" rpy="0 0 0"/>
     <axis xyz="0 0 1"/>
     <limit velocity="6.5" effort="1000" lower="${-pi*0.5}" upper="${pi*0.5}" />
@@ -99,5 +99,5 @@
   <link name="link4">
     <visual>
-      <origin xyz="0 0 0" rpy="${pi/2} 0 ${pi/2}"/>
+      <origin xyz="0 0 0" rpy="0 0 0"/>
       <geometry>
         <mesh filename="package://open_manipulator_7dof_description/meshes/link4.stl" scale="0.001 0.001 0.001"/>
@@ -106,5 +106,5 @@
     </visual>
     <collision>
-      <origin xyz="0 0 0" rpy="${pi/2} 0 ${pi/2}"/>
+      <origin xyz="0 0 0" rpy="0 0 0"/>
       <geometry>
         <mesh filename="package://open_manipulator_7dof_description/meshes/link4.stl" scale="0.001 0.001 0.001"/>
@@ -123,5 +123,5 @@
     <parent link="link4"/>
     <child link="link5"/>
-    <origin xyz="0.0 0.0 0.069" rpy="0 0 0"/>
+    <origin xyz="0.029998 0.05750 0.097498" rpy="0 0 0"/>
     <axis xyz="0 1 0"/>
     <limit velocity="6.5" effort="1000" lower="${-pi*0.5}" upper="${pi*0.5}" />
@@ -131,5 +131,5 @@
   <link name="link5">
     <visual>
-      <origin xyz="0 -0.057 0" rpy="${pi/2} 0 ${pi/2}"/>
+      <origin xyz="0 0 0" rpy="0 0 0"/>
       <geometry>
         <mesh filename="package://open_manipulator_7dof_description/meshes/link5.stl" scale="0.001 0.001 0.001"/>
@@ -138,5 +138,5 @@
     </visual>
     <collision>
-      <origin xyz="0 -0.057 0" rpy="${pi/2} 0 ${pi/2}"/>
+      <origin xyz="0 0 0" rpy="0 0 0"/>
       <geometry>
         <mesh filename="package://open_manipulator_7dof_description/meshes/link5.stl" scale="0.001 0.001 0.001"/>
@@ -155,6 +155,6 @@
     <parent link="link5"/>
     <child link="link6"/>
-    <origin xyz="0.0 0.0 0.195" rpy="0 0 0"/>
-    <axis xyz="0 0 1"/>
+    <origin xyz="0.195 -0.05750 0.03" rpy="0 0 0"/>
+    <axis xyz="1 0 0"/>
     <limit velocity="6.5" effort="1000" lower="${-pi*0.5}" upper="${pi*0.5}" />
     <dynamics damping="0.7"/>
@@ -163,5 +163,5 @@
   <link name="link6">
     <visual>
-      <origin xyz="0 0 0" rpy="${pi/2} 0 ${pi/2}"/>
+      <origin xyz="0 0 0" rpy="0 0 0"/>
       <geometry>
         <mesh filename="package://open_manipulator_7dof_description/meshes/link6.stl" scale="0.001 0.001 0.001"/>
@@ -170,5 +170,5 @@
     </visual>
     <collision>
-      <origin xyz="0 0 0" rpy="${pi/2} 0 ${pi/2}"/>
+      <origin xyz="0 0 0" rpy="0 0 0"/>
       <geometry>
         <mesh filename="package://open_manipulator_7dof_description/meshes/link6.stl" scale="0.001 0.001 0.001"/>
@@ -187,5 +187,5 @@
     <parent link="link6"/>
     <child link="link7"/>
-    <origin xyz="0.0 0.0 0.063" rpy="0 0 0"/>
+    <origin xyz="0.063 0.045 0.0" rpy="0 0 0"/>
     <axis xyz="0 1 0"/>
     <limit velocity="6.5" effort="1000" lower="${-pi*0.5}" upper="${pi*0.5}" />
@@ -195,5 +195,5 @@
   <link name="link7">
     <visual>
-      <origin xyz="0 -0.045 0" rpy="${pi/2} 0 ${pi/2}"/>
+      <origin xyz="0 0 0" rpy="0 0 0"/>
       <geometry>
         <mesh filename="package://open_manipulator_7dof_description/meshes/link7.stl" scale="0.001 0.001 0.001"/>
@@ -202,5 +202,5 @@
     </visual>
     <collision>
-      <origin xyz="0 -0.045 0" rpy="${pi/2} 0 ${pi/2}"/>
+      <origin xyz="0 0 0" rpy="0 0 0"/>
       <geometry>
         <mesh filename="package://open_manipulator_7dof_description/meshes/link7.stl" scale="0.001 0.001 0.001"/>
@@ -219,6 +219,6 @@
     <parent link="link7"/>
     <child link="end_link"/>
-    <origin xyz="0.0 0.0 0.12300" rpy="0 0 0"/>
-    <axis xyz="0 0 1"/>
+    <origin xyz="0.1230 -0.045 0.0" rpy="0 0 0"/>
+    <axis xyz="1 0 0"/>
     <limit velocity="6.5" effort="1000" lower="${-pi*0.5}" upper="${pi*0.5}" />
     <dynamics damping="0.7"/>
@@ -227,5 +227,5 @@
   <link name="end_link">
     <visual>
-      <origin xyz="0.0 0.0 0.0" rpy="0 -${pi/2} -${pi/2}" />
+      <origin xyz="0.0 0.0 0.0" rpy="0 0 0" />
       <geometry>
         <mesh filename="package://open_manipulator_7dof_description/meshes/end_link.stl" scale="0.001 0.001 0.001"/>
@@ -234,5 +234,5 @@
     </visual>
     <collision>
-      <origin xyz="0.0 0.0 0.0" rpy="0 -${pi/2} -${pi/2}" />
+      <origin xyz="0.0 0.0 0.0" rpy="0 0 0" />
       <geometry>
         <mesh filename="package://open_manipulator_7dof_description/meshes/end_link.stl" scale="0.001 0.001 0.001"/>

File: open_manipulator_7dof_description/urdf/open_manipulator_7dof_with_gripper.urdf.xacro (robot description, xacro)
@@ -4,5 +4,5 @@
   <link name="link1">
     <visual>
-      <origin xyz="0 0 0" rpy="${pi/2} 0 ${pi/2}"/>
+      <origin xyz="0 0 0" rpy="0 0 0"/>
       <geometry>
         <mesh filename="package://open_manipulator_7dof_description/meshes/link1.stl" scale="0.001 0.001 0.001"/>
@@ -11,5 +11,5 @@
     </visual>
     <collision>
-      <origin xyz="0 0 0" rpy="${pi/2} 0 ${pi/2}"/>
+      <origin xyz="0 0 0" rpy="0 0 0"/>
       <geometry>
         <mesh filename="package://open_manipulator_7dof_description/meshes/link1.stl" scale="0.001 0.001 0.001"/>
@@ -27,5 +27,5 @@
     <parent link="link1"/>
     <child link="link2"/>
-    <origin xyz="0.0 0.0 0.124" rpy="0 0 0"/>
+    <origin xyz="0.0 0.0 0.126" rpy="0 0 0"/>
     <axis xyz="0 0 1"/>
     <limit velocity="6.5" effort="1000" lower="${-pi*0.5}" upper="${pi*0.5}" />
@@ -35,5 +35,5 @@
   <link name="link2">
     <visual>
-      <origin xyz="0 0 0" rpy="${pi/2} 0 ${pi/2}"/>
+      <origin xyz="0 0 0" rpy="0 0 0"/>
       <geometry>
         <mesh filename="package://open_manipulator_7dof_description/meshes/link2.stl" scale="0.001 0.001 0.001"/>
@@ -42,5 +42,5 @@
     </visual>
     <collision>
-      <origin xyz="0 0 0" rpy="${pi/2} 0 ${pi/2}"/>
+      <origin xyz="0 0 0" rpy="0 0 0"/>
       <geometry>
         <mesh filename="package://open_manipulator_7dof_description/meshes/link2.stl" scale="0.001 0.001 0.001"/>
@@ -59,5 +59,5 @@
     <parent link="link2"/>
     <child link="link3"/>
-    <origin xyz="0.0 0.0 0.033" rpy="0 0 0"/>
+    <origin xyz="0.0 0.069 0.033" rpy="0 0 0"/>
     <axis xyz="0 1 0"/>
     <limit velocity="6.5" effort="1000" lower="${-pi*0.5}" upper="${pi*0.5}" />
@@ -67,5 +67,5 @@
   <link name="link3">
     <visual>
-      <origin xyz="0 -0.069 0.0" rpy="${pi/2} 0 ${pi/2}"/>
+      <origin xyz="0 0 0" rpy="0 0 0"/>
       <geometry>
         <mesh filename="package://open_manipulator_7dof_description/meshes/link3.stl" scale="0.001 0.001 0.001"/>
@@ -74,5 +74,5 @@
     </visual>
     <collision>
-      <origin xyz="0 -0.069 0.0" rpy="${pi/2} 0 ${pi/2}"/>
+      <origin xyz="0 0 0" rpy="0 0 0"/>
       <geometry>
         <mesh filename="package://open_manipulator_7dof_description/meshes/link3.stl" scale="0.001 0.001 0.001"/>
@@ -91,5 +91,5 @@
     <parent link="link3"/>
     <child link="link4"/>
-    <origin xyz="0.0 0.0 0.195" rpy="0 0 0"/>
+    <origin xyz="0.0 -0.069 0.195" rpy="0 0 0"/>
     <axis xyz="0 0 1"/>
     <limit velocity="6.5" effort="1000" lower="${-pi*0.5}" upper="${pi*0.5}" />
@@ -99,5 +99,5 @@
   <link name="link4">
     <visual>
-      <origin xyz="0 0 0" rpy="${pi/2} 0 ${pi/2}"/>
+      <origin xyz="0 0 0" rpy="0 0 0"/>
       <geometry>
         <mesh filename="package://open_manipulator_7dof_description/meshes/link4.stl" scale="0.001 0.001 0.001"/>
@@ -106,5 +106,5 @@
     </visual>
     <collision>
-      <origin xyz="0 0 0" rpy="${pi/2} 0 ${pi/2}"/>
+      <origin xyz="0 0 0" rpy="0 0 0"/>
       <geometry>
         <mesh filename="package://open_manipulator_7dof_description/meshes/link4.stl" scale="0.001 0.001 0.001"/>
@@ -123,5 +123,5 @@
     <parent link="link4"/>
     <child link="link5"/>
-    <origin xyz="0.0 0.0 0.069" rpy="0 0 0"/>
+    <origin xyz="0.029998 0.05750 0.097498" rpy="0 0 0"/>
     <axis xyz="0 1 0"/>
     <limit velocity="6.5" effort="1000" lower="${-pi*0.5}" upper="${pi*0.5}" />
@@ -131,5 +131,5 @@
   <link name="link5">
     <visual>
-      <origin xyz="0 -0.057 0" rpy="${pi/2} 0 ${pi/2}"/>
+      <origin xyz="0 0 0" rpy="0 0 0"/>
       <geometry>
         <mesh filename="package://open_manipulator_7dof_description/meshes/link5.stl" scale="0.001 0.001 0.001"/>
@@ -138,5 +138,5 @@
     </visual>
     <collision>
-      <origin xyz="0 -0.057 0" rpy="${pi/2} 0 ${pi/2}"/>
+      <origin xyz="0 0 0" rpy="0 0 0"/>
       <geometry>
         <mesh filename="package://open_manipulator_7dof_description/meshes/link5.stl" scale="0.001 0.001 0.001"/>
@@ -155,6 +155,6 @@
     <parent link="link5"/>
     <child link="link6"/>
-    <origin xyz="0.0 0.0 0.195" rpy="0 0 0"/>
-    <axis xyz="0 0 1"/>
+    <origin xyz="0.195 -0.05750 0.03" rpy="0 0 0"/>
+    <axis xyz="1 0 0"/>
     <limit velocity="6.5" effort="1000" lower="${-pi*0.5}" upper="${pi*0.5}" />
     <dynamics damping="0.7"/>
@@ -163,5 +163,5 @@
   <link name="link6">
     <visual>
-      <origin xyz="0 0 0" rpy="${pi/2} 0 ${pi/2}"/>
+      <origin xyz="0 0 0" rpy="0 0 0"/>
       <geometry>
         <mesh filename="package://open_manipulator_7dof_description/meshes/link6.stl" scale="0.001 0.001 0.001"/>
@@ -170,5 +170,5 @@
     </visual>
     <collision>
-      <origin xyz="0 0 0" rpy="${pi/2} 0 ${pi/2}"/>
+      <origin xyz="0 0 0" rpy="0 0 0"/>
       <geometry>
         <mesh filename="package://open_manipulator_7dof_description/meshes/link6.stl" scale="0.001 0.001 0.001"/>
@@ -187,5 +187,5 @@
     <parent link="link6"/>
     <child link="link7"/>
-    <origin xyz="0.0 0.0 0.063" rpy="0 0 0"/>
+    <origin xyz="0.063 0.045 0.0" rpy="0 0 0"/>
     <axis xyz="0 1 0"/>
     <limit velocity="6.5" effort="1000" lower="${-pi*0.5}" upper="${pi*0.5}" />
@@ -195,5 +195,5 @@
   <link name="link7">
     <visual>
-      <origin xyz="0 -0.045 0" rpy="${pi/2} 0 ${pi/2}"/>
+      <origin xyz="0 0 0" rpy="0 0 0"/>
       <geometry>
         <mesh filename="package://open_manipulator_7dof_description/meshes/link7.stl" scale="0.001 0.001 0.001"/>
@@ -202,5 +202,5 @@
     </visual>
     <collision>
-      <origin xyz="0 -0.045 0" rpy="${pi/2} 0 ${pi/2}"/>
+      <origin xyz="0 0 0" rpy="0 0 0"/>
       <geometry>
         <mesh filename="package://open_manipulator_7dof_description/meshes/link7.stl" scale="0.001 0.001 0.001"/>
@@ -219,6 +219,6 @@
     <parent link="link7"/>
     <child link="end_link"/>
-    <origin xyz="0.0 0.0 0.12300" rpy="0 0 0"/>
-    <axis xyz="0 0 1"/>
+    <origin xyz="0.1230 -0.045 0.0" rpy="0 0 0"/>
+    <axis xyz="1 0 0"/>
     <limit velocity="6.5" effort="1000" lower="${-pi*0.5}" upper="${pi*0.5}" />
     <dynamics damping="0.7"/>
@@ -227,5 +227,5 @@
   <link name="end_link">
     <visual>
-      <origin xyz="0.0 0.0 0.0" rpy="0 -${pi/2} -${pi/2}" />
+      <origin xyz="0.0 0.0 0.0" rpy="0 0 0" />
       <geometry>
         <mesh filename="package://open_manipulator_7dof_description/meshes/end_link.stl" scale="0.001 0.001 0.001"/>
@@ -234,5 +234,5 @@
     </visual>
     <collision>
-      <origin xyz="0.0 0.0 0.0" rpy="0 -${pi/2} -${pi/2}" />
+      <origin xyz="0.0 0.0 0.0" rpy="0 0 0" />
       <geometry>
         <mesh filename="package://open_manipulator_7dof_description/meshes/end_link.stl" scale="0.001 0.001 0.001"/>
@@ -250,5 +250,5 @@
     <parent link="end_link"/>
     <child link="gripper_main_link"/>
-    <origin xyz="0.0 0.0 0.00625" rpy="0 -${pi/2} 0" />
+    <origin xyz="0.007 0.0 0.0" rpy="0 0 0" />
   </joint>
   <!-- gripper main link -->

Commit message: update

File: open_manipulator_7dof_description/urdf/open_manipulator_7dof.urdf.xacro (robot description, xacro)
@@ -1,4 +1,5 @@
 <?xml version="1.0"?>
 <robot xmlns:xacro="http://www.ros.org/wiki/xacro">
+  <xacro:property name="leftarm_rightarm" default="${pi/2}"/>
   <!-- link 1 -->
   <link name="link1">
@@ -29,5 +30,5 @@
     <origin xyz="0.0 0.0 0.126" rpy="0 0 0"/>
     <axis xyz="0 0 1"/>
-    <limit velocity="6.5" effort="1000" lower="${-pi*0.5}" upper="${pi*0.5}" />
+    <limit velocity="6.5" effort="1000" lower="${-pi*0.95}" upper="${pi*0.95}" />
     <dynamics damping="0.7"/>
   </joint>
@@ -91,7 +92,7 @@
     <parent link="link3"/>
     <child link="link4"/>
-    <origin xyz="0.0 -0.069 0.195" rpy="0 0 0"/>
+    <origin xyz="0.0 -0.069 0.195" rpy="0 0 ${leftarm_rightarm}"/>
     <axis xyz="0 0 1"/>
-    <limit velocity="6.5" effort="1000" lower="${-pi*0.5}" upper="${pi*0.5}" />
+    <limit velocity="6.5" effort="1000" lower="${-pi*0.75}" upper="${pi*0.75}" />
     <dynamics damping="0.7"/>
   </joint>
@@ -125,5 +126,5 @@
     <origin xyz="0.029998 0.05750 0.097498" rpy="0 0 0"/>
     <axis xyz="0 1 0"/>
-    <limit velocity="6.5" effort="1000" lower="${-pi*0.5}" upper="${pi*0.5}" />
+    <limit velocity="6.5" effort="1000" lower="${-pi*0.65}" upper="${pi*0.5}" />
     <dynamics damping="0.7"/>
   </joint>
@@ -157,5 +158,5 @@
     <origin xyz="0.195 -0.05750 0.03" rpy="0 0 0"/>
     <axis xyz="1 0 0"/>
-    <limit velocity="6.5" effort="1000" lower="${-pi*0.5}" upper="${pi*0.5}" />
+    <limit velocity="6.5" effort="1000" lower="${-pi*0.95}" upper="${pi*0.95}" />
     <dynamics damping="0.7"/>
   </joint>
@@ -218,25 +219,25 @@
   <joint name="joint7" type="revolute">
     <parent link="link7"/>
-    <child link="end_link"/>
+    <child link="fake_end_link"/>
     <origin xyz="0.1230 -0.045 0.0" rpy="0 0 0"/>
     <axis xyz="1 0 0"/>
-    <limit velocity="6.5" effort="1000" lower="${-pi*0.5}" upper="${pi*0.5}" />
+    <limit velocity="6.5" effort="1000" lower="${-pi*0.95}" upper="${pi*0.95}" />
     <dynamics damping="0.7"/>
   </joint>
   <!-- end link -->
-  <link name="end_link">
-    <visual>
+  <link name="fake_end_link">
+    <visual>
+      <origin xyz="0.0 0.0 0.0" rpy="0 0 0" />
+      <geometry>
+        <box size="0.01 0.01 0.01"/>
+      </geometry>
+      <material name="grey"/>
+    </visual>
+    <!-- <collision>
       <origin xyz="0.0 0.0 0.0" rpy="0 0 0" />
       <geometry>
         <mesh filename="package://open_manipulator_7dof_description/meshes/end_link.stl" scale="0.001 0.001 0.001"/>
       </geometry>
-      <material name="grey"/>
-    </visual>
-    <collision>
-      <origin xyz="0.0 0.0 0.0" rpy="0 0 0" />
-      <geometry>
-        <mesh filename="package://open_manipulator_7dof_description/meshes/end_link.stl" scale="0.001 0.001 0.001"/>
-      </geometry>
-    </collision>
+    </collision> -->
     <inertial>
       <origin xyz="0.00337 0.00000 0.00000" rpy="0 0 0"/>
@@ -246,3 +247,25 @@
     </inertial>
   </link>
+  <!-- end link -->
+  <!-- <link name="end_link">
+    <visual>
+      <origin xyz="0.0 0.0 0.0" rpy="0 0 0" />
+      <geometry>
+        <mesh filename="package://open_manipulator_7dof_description/meshes/end_link.stl" scale="0.001 0.001 0.001"/>
+      </geometry>
+      <material name="grey"/>
+    </visual>
+    <collision>
+      <origin xyz="0.0 0.0 0.0" rpy="0 0 0" />
+      <geometry>
+        <mesh filename="package://open_manipulator_7dof_description/meshes/end_link.stl" scale="0.001 0.001 0.001"/>
+      </geometry>
+    </collision>
+    <inertial>
+      <origin xyz="0.00337 0.00000 0.00000" rpy="0 0 0"/>
+      <mass value="0.01919"/>
+      <inertia ixx="1.0" ixy="0.0" ixz="0.0" iyy="1.0" iyz="0.0" izz="1.0" />
+      <!-<inertia ixx="0.00000938" ixy="0.0" ixz="0.0" iyy="0.00000338" iyz="0.0" izz="0.00000635" />->
+    </inertial>
+  </link> -->
 </robot>

File: open_manipulator_7dof_description/urdf/open_manipulator_7dof_robot.urdf (robot description, URDF)
Before this commit: robot open_manipulator_7dof, 8 links, 7 joints
Links:
- removed link end_link
- added link fake_end_link, mass 0.01919; visual box size=0.01 0.01 0.01
Joints:
- joint joint1: limit lower=-1.57079632679 upper=1.57079632679 effort=1000 velocity=6.5 -> lower=-2.98451302091 upper=2.98451302091 effort=1000 velocity=6.5; origin xyz=0.0 0.0 0.124 rpy=0 0 0 -> xyz=0.0 0.0 0.126 rpy=0 0 0
- joint joint2: origin xyz=0.0 0.0 0.033 rpy=0 0 0 -> xyz=0.0 0.069 0.033 rpy=0 0 0
- joint joint3: limit lower=-1.57079632679 upper=1.57079632679 effort=1000 velocity=6.5 -> lower=-2.35619449019 upper=2.35619449019 effort=1000 velocity=6.5; origin xyz=0.0 0.0 0.195 rpy=0 0 0 -> xyz=0.0 -0.069 0.195 rpy=0 0 0
- joint joint4: limit lower=-1.57079632679 upper=1.57079632679 effort=1000 velocity=6.5 -> lower=-2.04203522483 upper=1.57079632679 effort=1000 velocity=6.5; origin xyz=0.0 0.0 0.069 rpy=0 0 0 -> xyz=0.029998 0.05750 0.097498 rpy=0 0 0
- joint joint5: axis 0 0 1 -> 1 0 0; limit lower=-1.57079632679 upper=1.57079632679 effort=1000 velocity=6.5 -> lower=-2.98451302091 upper=2.98451302091 effort=1000 velocity=6.5; origin xyz=0.0 0.0 0.195 rpy=0 0 0 -> xyz=0.195 -0.05750 0.03 rpy=0 0 0
- joint joint6: origin xyz=0.0 0.0 0.063 rpy=0 0 0 -> xyz=0.063 0.045 0.0 rpy=0 0 0
- joint joint7: axis 0 0 1 -> 1 0 0; child end_link -> fake_end_link; limit lower=-1.57079632679 upper=1.57079632679 effort=1000 velocity=6.5 -> lower=-2.98451302091 upper=2.98451302091 effort=1000 velocity=6.5; origin xyz=0.0 0.0 0.12300 rpy=0 0 0 -> xyz=0.1230 -0.045 0.0 rpy=0 0 0

File: open_manipulator_7dof_description/urdf/open_manipulator_7dof_robot.urdf.xacro (robot description, xacro)
@@ -1,4 +1,5 @@
 <?xml version="1.0"?>
 <robot name="open_manipulator_7dof" xmlns:xacro="http://www.ros.org/wiki/xacro">
+  <xacro:property name="leftarm_rightarm" default="${pi/2}"/>
   <!-- Import Rviz colors -->
   <xacro:include filename="$(find open_manipulator_7dof_description)/urdf/materials.xacro" />
@@ -10,10 +11,10 @@
   <xacro:include filename="$(find open_manipulator_7dof_description)/urdf/open_manipulator_7dof.urdf.xacro" />
   <!-- World -->
-  <link name="world"/>
+  <!-- <link name="world"/> -->
   <!-- World fixed joint-->
-  <joint name="world_fixed" type="fixed">
+  <!-- <joint name="world_fixed" type="fixed">
     <origin xyz="0 0 0" rpy="0 0 0"/>
     <parent link="world"/>
     <child link="link1"/>
-  </joint>
+  </joint> -->
 </robot>
