Commit message: update

File: open_manipulator_7dof_description/urdf/open_manipulator_7dof.gazebo.xacro (robot description, xacro)
@@ -30,5 +30,5 @@
   <RefLink ref="link7"/>
   <!-- end_link -->
-  <RefLink ref="end_link"/>
+  <RefLink ref="fake_end_link"/>
   <!-- ros_control plugin -->
   <gazebo>

File: open_manipulator_7dof_description/urdf/open_manipulator_7dof.urdf.xacro (robot description, xacro)
@@ -1,5 +1,12 @@
 <?xml version="1.0"?>
 <robot xmlns:xacro="http://www.ros.org/wiki/xacro">
-  <xacro:property name="leftarm_rightarm" default="${pi/2}"/>
+  <!-- Left or Right configuration -->
+  <xacro:property name="left_right" default="left"/>
+  <xacro:if value="${left_right == 'left'}">
+    <xacro:property name="leftarm_rightarm" default="-${pi/2}"/>
+  </xacro:if>
+  <xacro:if value="${left_right == 'right'}">
+    <xacro:property name="leftarm_rightarm" default="${pi/2}"/>
+  </xacro:if>
   <!-- link 1 -->
   <link name="link1">

File: open_manipulator_7dof_description/urdf/open_manipulator_7dof_robot.urdf (robot description, URDF)
Before this commit: robot open_manipulator_7dof, 8 links, 7 joints
Links:
- added link world
Joints:
- added joint world_fixed: type fixed, parent world, child link1, origin xyz=0 0 0 rpy=0 0 0
- joint joint3: origin xyz=0.0 -0.069 0.195 rpy=0 0 0 -> xyz=0.0 -0.069 0.195 rpy=0 0 1.57079632679

File: open_manipulator_7dof_description/urdf/open_manipulator_7dof_robot.urdf.xacro (robot description, xacro)
@@ -1,5 +1,6 @@
 <?xml version="1.0"?>
 <robot name="open_manipulator_7dof" xmlns:xacro="http://www.ros.org/wiki/xacro">
-  <xacro:property name="leftarm_rightarm" default="${pi/2}"/>
+  <!-- Left or Right configuration -->
+  <xacro:property name="left_right" default="left"/>
   <!-- Import Rviz colors -->
   <xacro:include filename="$(find open_manipulator_7dof_description)/urdf/materials.xacro" />
@@ -11,10 +12,10 @@
   <xacro:include filename="$(find open_manipulator_7dof_description)/urdf/open_manipulator_7dof.urdf.xacro" />
   <!-- World -->
-  <!-- <link name="world"/> -->
+  <link name="world"/>
   <!-- World fixed joint-->
-  <!-- <joint name="world_fixed" type="fixed">
+  <joint name="world_fixed" type="fixed">
     <origin xyz="0 0 0" rpy="0 0 0"/>
     <parent link="world"/>
     <child link="link1"/>
-  </joint> -->
+  </joint>
 </robot>
